File: hardware/pcb/layout/kicad/dotglow-v1.kicad_pcb (KiCad board)
At the start: 2 copper layers, 128 x 33 mm, 41 parts, among them J1 USB-C 5V, J2 DISPLAY IN, J3 DHT22, J4 I2C (RTC V2), J5 SPEAKER 8R 2W, J6 LDR, J7 STOPWATCH SW, SW1 RESET, SW2 BOOT, SW3 STOPWATCH, U1 ESP32-S3-MINI-1-N8, U2 AP2112K-3.3, U3 74AHCT125, U4 MAX98357A, U5 USBLC6-2SC6

Commit message: DotGlow V1 board: switch to ESP32-S3-WROOM-1-N16R8 (C2913202), full pinout doc, display header on the module end, rebuild script
Co-Authored-By: ElectroIoT <electroiot.in@gmail.com>
Parts:
- U1: value ESP32-S3-MINI-1-N8 -> ESP32-S3-WROOM-1-N16R8; footprint RF_Module:ESP32-S2-MINI-1 -> RF_Module:ESP32-S3-WROOM-1
- moved J5 4.00 mm to (120.0, 75.0)
- moved J7 4.00 mm to (111.0, 77.0)
- moved SW1 4.00 mm to (84.0, 77.0)
- moved SW2 4.00 mm to (94.0, 77.0)
- moved SW3 4.00 mm to (104.0, 77.0)
- moved TP1 4.00 mm to (127.0, 77.0)
- moved TP2 4.00 mm to (131.0, 77.0)
- moved J2 3.53 mm to (175.5, 61.4)
- moved R1 3.20 mm to (80.0, 64.5)
- moved C4 2.83 mm to (80.0, 69.0)
- moved U1 2.50 mm to (62.8, 66.5)
Connections:
- U1 pad 10: I2S_LRC -> unconnected-(U1-IO17-Pad10)
- U1 pad 11: I2S_DIN -> unconnected-(U1-IO18-Pad11)
- U1 pad 13: I2C_SCL -> USB_DN
- U1 pad 14: MAX_CS_3V -> USB_DP
- U1 pad 15: MAX_DIN_3V -> unconnected-(U1-IO3-Pad15)
- U1 pad 16: MAX_CLK_3V -> unconnected-(U1-IO46-Pad16)
- U1 pad 17: DHT_DATA -> I2C_SCL
- U1 pad 18: unconnected-(U1-IO14-Pad18) -> MAX_CS_3V
- U1 pad 19: AMP_SD -> MAX_DIN_3V
- U1 pad 2: GND -> +3V3
- U1 pad 20: unconnected-(U1-IO16-Pad20) -> MAX_CLK_3V
- U1 pad 21: unconnected-(U1-IO17-Pad21) -> DHT_DATA
- U1 pad 23: USB_DN -> unconnected-(U1-IO21-Pad23)
- U1 pad 24: USB_DP -> unconnected-(U1-IO47-Pad24)
- U1 pad 27: unconnected-(U1-IO47-Pad27) -> BOOT
- U1 pad 3: +3V3 -> EN
- U1 pad 38: unconnected-(U1-IO42-Pad38) -> NTC_ADC
- U1 pad 39: unconnected-(U1-TXD0-Pad39) -> LDR_ADC
- U1 pad 4: BOOT -> STOPWATCH
- U1 pad 40: unconnected-(U1-RXD0-Pad40) -> GND
- U1 pad 41: unconnected-(U1-IO45-Pad41) -> GND
- U1 pad 5: LDR_ADC -> I2S_BCLK
- U1 pad 6: NTC_ADC -> I2S_LRC
- U1 pad 7: unconnected-(U1-IO3-Pad7) -> I2S_DIN
- U1 pad 8: STOPWATCH -> AMP_SD
- U1 pad 9: I2S_BCLK -> unconnected-(U1-IO16-Pad9)

Commit message: DotGlow V1 board: JST XA connectors (2-pin C265077, 3-pin C265055, 4-pin C491709) for speaker, stopwatch, LDR, DHT22, I2C; re-placed and re-routed
Co-Authored-By: ElectroIoT <electroiot.in@gmail.com>
Parts:
- J3: footprint Connector_PinHeader_2.54mm:PinHeader_1x03_P2.54mm_Vertical -> Connector_JST:JST_XA_B03B-XASK-1_1x03_P2.50mm_Vertical
- J4: footprint Connector_PinHeader_2.54mm:PinHeader_1x04_P2.54mm_Vertical -> Connector_JST:JST_XA_B04B-XASK-1-A_1x04_P2.50mm_Vertical
- J5: footprint Connector_JST:JST_PH_S2B-PH-K_1x02_P2.00mm_Horizontal -> Connector_JST:JST_XA_B02B-XASK-1-A_1x02_P2.50mm_Vertical
- J6, J7: footprint Connector_PinHeader_2.54mm:PinHeader_1x02_P2.54mm_Vertical -> Connector_JST:JST_XA_B02B-XASK-1-A_1x02_P2.50mm_Vertical
- moved J6 15.5 mm to (141.0, 77.5)
- moved J3 8.00 mm to (156.0, 67.0)
- moved J4 5.10 mm to (142.0, 67.0)
- moved TP1 3.00 mm to (130.0, 77.0)
- moved TP2 3.00 mm to (134.0, 77.0)
- moved J5 2.92 mm to (121.5, 77.5)
- moved U5 2.06 mm to (150.0, 76.5)
- moved J7 1.58 mm to (112.5, 77.5)
- moved R10 1.00 mm to (168.0, 72.0)
- moved R9 1.00 mm to (165.0, 72.0)

Commit message: DotGlow V1 board: final EasyEDA files (schematic, PCB, BOM, Gerber), 3D renders and viewer angles, README banner, HyperFrames short video source
Co-Authored-By: ElectroIoT <electroiot.in@gmail.com>
Parts:
- U2: value AP2112K-3.3 -> XC6220B331MR-G
